Commit message: merge_file

File: src/my_robot_description/urdf/camera.xacro (robot description, xacro)
@@ -12,10 +12,10 @@
                     <format>R8G8B8</format>
                 </image>
-                    <clip>
+                <clip>
                     <near>0.02</near>
                     <far>300</far>
                 </clip>
                 <noise>
-                    <type>gaussian</type>
+                <type>gaussian</type>
                     <mean>0.0</mean>
                     <stddev>0.01</stddev>
@@ -23,6 +23,6 @@
             </camera>
             <plugin name="camera_controller" filename="libgazebo_ros_camera.so">
-            <frame_name>camera_link</frame_name>
-            <hack_baseline>0.07</hack_baseline>
+                <frame_name>camera_link</frame_name>
+                <hack_baseline>0.07</hack_baseline>
             </plugin>
         </sensor>

File: src/my_robot_description/urdf/lidar.xacro (robot description, xacro)
@@ -2,36 +2,36 @@
 <robot xmlns:xacro="http://www.ros.org/wiki/xacro" >
     <gazebo reference="laser_link">
-    <sensor name="laser" type="ray">
-        <pose>0 0 0 0 0 0</pose>
-        <always_on>1</always_on>
-        <update_rate>15</update_rate>
-        <visualize>true</visualize>
-        <ray>
-            <scan>
-                <horizontal>
-                    <samples>375</samples>
-                    <resolution>1</resolution>
-                    <min_angle>${-180*pi/180}</min_angle>
-                    <max_angle>${180*pi/180}</max_angle>
-                </horizontal>
-            </scan>
-            <range>
-                <min>0.12</min>
-                <max>8.0</max>
-                <resolution>0.05</resolution>
-            </range>
-            <noise>
-                <type>gaussian</type>
-                <mean>0.0</mean>
-                <stddev>0.01</stddev>
-            </noise>
-        </ray>
-        <plugin name="laser" filename="libgazebo_ros_ray_sensor.so">
-            <ros>
-                <remapping>~/out:=scan</remapping>
-            </ros>
-            <frame_name>laser_link</frame_name>
-            <output_type>sensor_msgs/LaserScan</output_type>
-        </plugin>
+        <sensor name="laser" type="ray">
+            <pose>0 0 0 0 0 0</pose>
+            <always_on>1</always_on>
+            <update_rate>15</update_rate>
+            <visualize>false</visualize>
+            <ray>
+                <scan>
+                    <horizontal>
+                        <samples>375</samples>
+                        <resolution>1</resolution>
+                        <min_angle>${-180*pi/180}</min_angle>
+                        <max_angle>${180*pi/180}</max_angle>
+                    </horizontal>
+                </scan>
+                <range>
+                    <min>0.12</min>
+                    <max>8.0</max>
+                    <resolution>0.05</resolution>
+                </range>
+                <noise>
+                    <type>gaussian</type>
+                    <mean>0.0</mean>
+                    <stddev>0.01</stddev>
+                </noise>
+            </ray>
+            <plugin name="laser" filename="libgazebo_ros_ray_sensor.so">
+                <ros>
+                    <remapping>~/out:=scan</remapping>
+                </ros>
+                <frame_name>laser_link</frame_name>
+                <output_type>sensor_msgs/LaserScan</output_type>
+            </plugin>
         </sensor>
     </gazebo>

File: src/my_robot_description/urdf/robot.urdf.xacro (robot description, xacro)
@@ -1,9 +1,8 @@
 <?xml version="1.0"?>
-<robot name="SLAM_repo" xmlns:xacro="http://www.ros.org/wiki/xacro">
+<robot name="my_mobile" xmlns:xacro="http://www.ros.org/wiki/xacro">
     <xacro:include filename="robot_core.xacro"/>
     <xacro:include filename="robot_gazebo.xacro"/>
-    <!-- <xacro:include filename="gazebo_control.xacro"/> -->
     <xacro:include filename="ros2_control.xacro" />
     <xacro:include filename="lidar.xacro" />
-    <xacro:include filename="camera.xacro" />
+    <xacro:include filename="camera.xacro"/>
 </robot>

File: src/my_robot_description/urdf/robot_core.xacro (robot description, xacro)
@@ -1,4 +1,4 @@
 <?xml version="1.0"?>
-<robot name="SLAM_repo" xmlns:xacro="http://www.ros.org/wiki/xacro">
+<robot name="my_mobile" xmlns:xacro="http://www.ros.org/wiki/xacro">
     <xacro:property name="wheel_separation" value="0.180"/>
     <xacro:property name="wheel_diameter" value="0.068"/>
@@ -7,8 +7,8 @@
         <parent link="base_footprint"/>
         <child link="base_link"/>
-        <origin xyz="0 ${wheel_diameter/2} 0" rpy="0 0 0"/>
+        <origin xyz="0 0 ${wheel_diameter/2}" rpy="0 0 0"/>
     </joint>
-    <link name="base_link">
-        <visual>
+	<link name="base_link">
+		<visual>
             <origin xyz="0 0 0" rpy="0 0 0"/>
             <geometry>
@@ -27,5 +27,5 @@
             <inertia ixx="0.01" ixy="0" ixz="0" iyy="0.01" iyz="0" izz="0.01"/>
         </inertial>
-    </link>
+	</link>
     <joint name="left_wheel_joint" type="continuous">
         <parent link="base_link"/>
@@ -93,5 +93,5 @@
         <inertial>
             <origin xyz="0.005 0 0.013" rpy="0 0 0"/>
-            <mass value="0.05000"/>
+            <mass value="0.050000"/>
             <inertia ixx="0.000005" ixy="0" ixz="-0.000001" iyy="0.000004" iyz="0" izz="0.000003"/>
         </inertial>
@@ -108,5 +108,5 @@
         <origin xyz="0.02 0 0" rpy="0 0 0"/>
     </joint>
-    <link name="ydlidar_sensor_mount">
+    <link name="ydlidar_lidar_mount">
         <visual>
             <origin xyz="0 0 0" rpy="0 0 0"/>
@@ -122,17 +122,17 @@
         </collision>
         <inertial>
-            <origin xyz="0.007 0 0" rpy="0 0 0"/>
+            <origin xyz="0.007 0 0.025" rpy="0 0 0"/>
             <mass value="0.150"/>
-            <inertia ixx="0.000058" ixy="0" ixz="0.000005" iyy="0.0000099" iyz="0" izz="0.000103"/>
+            <inertia ixx="0.000058" ixy="0" ixz="0.000005" iyy="0.000099" iyz="0" izz="0.000103"/>
         </inertial>
     </link>
     <joint name="idar_mount_fixed_joint" type="fixed">
         <parent link="base_link"/>
-        <child link="ydlidar_sensor_mount"/>
+        <child link="ydlidar_lidar_mount"/>
         <origin xyz="-0.01 0 0.085" rpy="0 0 0"/>
     </joint>
     <link name="laser_link"/>
     <joint name="laser_link_fixed_joint" type="fixed">
-        <parent link="ydlidar_sensor_mount"/>
+        <parent link="ydlidar_lidar_mount"/>
         <child link="laser_link"/>
         <origin xyz="0 0 0.04245" rpy="0 0 0"/>

File: src/my_robot_description/urdf/robot_gazebo.xacro (robot description, xacro)
@@ -1,4 +1,4 @@
 <?xml version="1.0"?>
-<robot name="SLAM_repo" xmlns:xacro="http://www.ros.org/wiki/xacro">
+<robot name="my_mobile" xmlns:xacro="http://www.ros.org/wiki/xacro">
     <gazebo reference="left_wheel">
         <mu1>200</mu1>

File: src/my_robot_description/urdf/ros2_control.xacro (robot description, xacro)
@@ -25,8 +25,8 @@
         <plugin filename="libgazebo_ros2_control.so" name="gazebo_ros2_control">
             <parameters>$(find my_robot_gazebo)/config/my_controllers.yaml</parameters>
-        <ros>
-            <remapping>diff_cont/cmd_vel_unstamped:=cmd_vel</remapping>
-            <remapping>diff_cont/odom:=odom</remapping>
-        </ros>
+            <ros>
+                <remapping>diff_cont/cmd_vel_unstamped:=cmd_vel</remapping>
+                <remapping>diff_cont/odom:=odom</remapping>
+            </ros>
         </plugin>
     </gazebo>
